Commit message: Add X-rail as 6th DOF (prismatic rail_joint)
Extends the SO-101 with a linear X-axis: rail + carriage links and a
prismatic rail_joint in the URDF, registered in ros2_control, the arm
controller, and all MoveIt configs (SRDF planning group, joint limits,
collision exceptions). With 6 DOF, position_only_ik is disabled so full
6D poses are solvable; the web GUI gets rail_joint (meters), a world
reference frame, and editable roll/pitch/yaw targets. Adds
waypoint_runner.py for driving 6D Cartesian waypoint sequences via
MoveIt IK, plus a diary entry noting the rail URDF geometry is
approximate and needs a revision for a fully realistic assembly.

Co-Authored-By: Claude Fable 5 <noreply@anthropic.com>

File: lerobot/src/lerobot_description/urdf/so101_base.xacro (robot description, xacro)
@@ -8,8 +8,82 @@
 	<!-- Links -->
 	<link name="world" />
+	<!-- ===================== X-Linearachse (6. DOF) ===================== -->
+	<!-- Statische Schiene (fest mit der Welt verbunden) -->
+	<link name="rail_link">
+		<!-- Rail 1. rpy dreht die Mesh-Laenge (Z) auf Welt-X; xyz zentriert die
+		     1 m lange Schiene um den Fahrweg und legt sie unter die Platte.
+		     Feinjustage in RViz. -->
+		<visual>
+			<origin xyz="-0.5 0 -0.085" rpy="1.5708 0 1.5708" />
+			<geometry>
+				<mesh filename="package://lerobot_description/meshes/rail/rail.stl"
+					scale="0.0001 0.0001 0.0001" />
+			</geometry>
+			<material name="3d_printed" />
+		</visual>
+		<!-- Rail 2, 90 mm in -Y versetzt -->
+		<visual>
+			<origin xyz="-0.5 -0.090 -0.085" rpy="1.5708 0 1.5708" />
+			<geometry>
+				<mesh filename="package://lerobot_description/meshes/rail/rail.stl"
+					scale="0.0001 0.0001 0.0001" />
+			</geometry>
+			<material name="3d_printed" />
+		</visual>
+		<inertial>
+			<origin xyz="0 0 0" rpy="0 0 0" />
+			<mass value="1.0" />
+			<inertia ixx="0.01" ixy="0" ixz="0" iyy="0.01" iyz="0" izz="0.01" />
+		</inertial>
+	</link>
+	<!-- z=0.085 hebt das Konstrukt an, damit die Rail-Unterkante (z=-0.085
+	     im rail-Frame) auf dem Gazebo-Boden (z=0) aufliegt statt darin zu
+	     versinken (vergrabene Kollisionsmeshes machen die Physik extrem langsam). -->
+	<joint name="world_to_rail" type="fixed">
+		<parent link="world" />
+		<child link="rail_link" />
+		<origin xyz="0 0 0.085" rpy="0 0 0" />
+	</joint>
+	<!-- Bewegter Schlitten (Platte + spaeter Slider) -->
+	<link name="carriage_link">
+		<!-- Platte 180 um Y gedreht (zeigt nach oben), dann zentriert:
+		     mittig in XY, Oberkante auf carriage-Frame. -->
+		<visual>
+			<origin xyz="0.070 -0.070 0" rpy="0 3.14159 0" />
+			<geometry>
+				<mesh filename="package://lerobot_description/meshes/rail/plate.stl"
+					scale="0.0001 0.0001 0.0001" />
+			</geometry>
+			<material name="3d_printed" />
+		</visual>
+		<inertial>
+			<origin xyz="0 0 0" rpy="0 0 0" />
+			<mass value="0.5" />
+			<inertia ixx="0.001" ixy="0" ixz="0" iyy="0.001" iyz="0" izz="0.001" />
+		</inertial>
+	</link>
+	<!-- Der neue 6. Freiheitsgrad: prismatisch entlang X -->
+	<joint name="rail_joint" type="prismatic">
+		<parent link="rail_link" />
+		<child link="carriage_link" />
+		<origin xyz="0 0 0" rpy="0 0 0" />
+		<axis xyz="1 0 0" />
+		<limit effort="50" velocity="1.0" lower="-0.5" upper="0.5" />
+	</joint>
+	<transmission name="rail_joint_trans">
+		<type>transmission_interface/SimpleTransmission</type>
+		<joint name="rail_joint">
+			<hardwareInterface>hardware_interface/PositionJointInterface</hardwareInterface>
+		</joint>
+		<actuator name="motor_rail">
+			<hardwareInterface>hardware_interface/PositionJointInterface</hardwareInterface>
+			<mechanicalReduction>1</mechanicalReduction>
+		</actuator>
+	</transmission>
+	<!-- Roboter sitzt auf der Platte. Feinjustage: 7 cm runter, 3 cm in -X. -->
 	<joint name="base_joint" type="fixed">
-		<parent link="world" />
+		<parent link="carriage_link" />
 		<child link="base" />
-		<origin xyz="0 0 0" rpy="0 0 0" />
+		<origin xyz="-0.03 0 -0.07" rpy="0 0 0" />
 	</joint>
 	<!-- Materials -->

File: lerobot/src/lerobot_description/urdf/so101_ros2_control.xacro (robot description, xacro)
@@ -14,4 +14,11 @@
             </xacro:unless>
         </hardware>
+        <joint name="rail_joint">
+            <command_interface name="position">
+                <param name="min">-0.5</param>
+                <param name="max">0.5</param>
+            </command_interface>
+            <state_interface name="position" />
+        </joint>
         <joint name="1">
             <command_interface name="position">

Commit message: Add TCP tool frame, startup script and task-space Home button
The gripper link frame comes from CAD with its X axis pointing straight up,
which forces pitch = -90 in the RPY decomposition. The setup was therefore
permanently parked in the gimbal-lock singularity: roll and yaw were ambiguous
(only their sum is defined), so the GUI displayed values far from what was
commanded even though the rotation was in fact identical.

Add a `tcp` link with the standard tool convention (Z = approach direction,
X horizontal) attached to `gripper` by a fixed joint. The approach direction was
derived from the jaw mesh geometry rather than guessed: the jaw extends to
gripper z = -0.105, so the gripper approaches along gripper -Z. GUI and
waypoint_runner now target `tcp`; `gripper_to_tcp` is part of the SRDF arm group
so MoveIt can solve IK for it. Round-trip verified: commanded RPY comes back
within 1 degree.

Also:
- start_rail.sh brings the rail setup up from a cold start and verifies each
  step (controllers active, /compute_ik available, rail_joint in /joint_states).
  It rebuilds first, because Gazebo spawns the robot from install/, and kills
  stale processes, because a surviving publisher serves the old robot
  description. Note the bracket trick in the pkill patterns - without it pkill
  matches its own shell and kills itself before the later lines run.
- rail_runner.py drives only the rail, without MoveIt.
- The task-space "Reset to 0" button becomes "Home" and fills in the pose the
  robot has with every joint at 0; resetting that section to 0/0/0 was
  meaningless. The values come from a single HOME_POSE constant injected into
  the page.
- moveit.rviz gains a TF display and its fixed frame changes from Base to
  world - with base as reference the world appeared to move whenever the rail
  travelled.

Co-Authored-By: Claude Opus 4.8 <noreply@anthropic.com>

File: lerobot/src/lerobot_description/urdf/so101_base.xacro (robot description, xacro)
@@ -413,4 +413,21 @@
 		</collision>
 	</link>
+	<!-- ===================== TCP (tool center point) =====================
+	     The `gripper` link frame comes from CAD and is awkward to command:
+	     its X axis points straight up in typical poses, which forces the
+	     RPY decomposition into pitch = -90 (gimbal lock) - roll and yaw then
+	     become ambiguous and the GUI shows different numbers than commanded.
+	     This frame fixes that by using the standard tool convention:
+	       TCP Z  = approach direction (out of the gripper, = gripper -Z)
+	       TCP X  = gripper +Y  (horizontal -> away from the singularity)
+	       TCP Y  = gripper +X
+	     Origin sits on the approach axis at the grasp point (fingertip is at
+	     gripper z = -0.105 m). Rotation rpy = (180deg, 0, 90deg). -->
+	<link name="tcp" />
+	<joint name="gripper_to_tcp" type="fixed">
+		<parent link="gripper" />
+		<child link="tcp" />
+		<origin xyz="0 0 -0.090" rpy="3.14159 0 1.5708" />
+	</joint>
 	<!-- Joint from gripper to jaw -->
 	<joint name="6" type="revolute">
